File: circuito v6.sch (EAGLE design)
At the start: 64 parts, among them IC1 LM324N

Commit message: Cambio de pines
Tras chequear lado izq y der de los phones, cambio los nombres de los pines para que queden
Estimulo Izq PIN 11
Estimulo Der PIN 12
Feedback Izq PIN 2
Feedback Der PIN 5
Ruido blanco Izq PIN 9
Ruido blanco Der PIN 10

Se reacomodan los pins, despues de renombrarlos, en sus posiciones correctas.
Se ripupea todo el routeo hecho.

Se creo esta branch porque eliminar los commits que se realizaron con estos mismos cambios pero no exitosamente, es no-trivial.
Parts:
- removed PIN13: (no value), pinhead:PINHD-1X1
- added PIN11: (no value), pinhead:PINHD-1X1
Connections:
- net N$16: now also PIN2.1; no longer PIN5.1
- net N$20: now also PIN11.1; no longer PIN9.1
- net N$21: now also PIN9.1; no longer PIN12.1
- net N$3: now also PIN12.1; no longer PIN13.1
- net N$7: now also PIN5.1; no longer PIN2.1
Other:
- note added: "Estimulo"
- note added: "Feedback con switch"
- note added: "Ruido blanco"
- moved on the sheet: PIN12, PIN2, PIN5, PIN9
